Commit message: Add minibot_gazebo package to display minibot model in Gazebo. Update mini_bot urdf to compatible with Gazebo.

File: mini_bot/urdf/mini_bot.urdf.xacro (robot description, xacro)
@@ -12,4 +12,14 @@
   <xacro:property name="mass5" value="0.24686"/> <!-- assumption value for mass -->
   <xacro:property name="mass6" value="0.024508"/> <!-- assumption value for mass -->
+  <!-- Import all Gazebo-customization elements, including Gazebo colors -->
+  <xacro:include filename="$(find mini_bot)/urdf/mini_bot.gazebo" />
+  <!-- Add a world link to fix rbot to Gazebo 'base_link' -->
+  <link name="world"/>
+  <joint name="fixed_base_joint" type="fixed">
+    <parent link="world"/>
+    <child link="base_link"/>
+    <origin xyz="0 0 0" rpy="0 0 0"/>
+  </joint>
+  <!-- Start the description of robot -->
   <link name="base_link">
     <inertial>
@@ -68,4 +78,5 @@
     <axis xyz="0 0 1" />
     <limit lower="-2.617993878" upper="3.019419606" effort="0" velocity="0" />
+    <dynamics damping="0.7"/>
   </joint>
   <link name="A2_Link">
@@ -101,4 +112,5 @@
     <axis xyz="0 0 1" />
     <limit lower="-1.6057029118" upper="1.9198621772" effort="0" velocity="0" />
+    <dynamics damping="0.7"/>
   </joint>
   <link name="A3_Link">
@@ -133,4 +145,5 @@
     <axis xyz="0 0 1" />
     <limit lower="-1.0821041362" upper="2.5307274154" effort="0" velocity="0" />
+    <dynamics damping="0.7"/>
   </joint>
   <link name="A4_Link">
@@ -165,4 +178,5 @@
     <axis xyz="0 0 1" />
     <limit lower="-2.0943951024" upper="3.0805061298" effort="0" velocity="0" />
+    <dynamics damping="0.7"/>
   </joint>
   <link name="A5_Link">
@@ -197,4 +211,5 @@
     <axis xyz="0 0 1" />
     <limit lower="-1.8325957146" upper="1.8325957146" effort="0" velocity="0" />
+    <dynamics damping="0.7"/>
   </joint>
   <link name="A6_Link">
@@ -229,4 +244,66 @@
     <axis xyz="0 0 1" />
     <limit lower="-3.1415926536" upper="3.1415926536" effort="0" velocity="0" />
-  </joint>
+    <dynamics damping="0.7"/>
+  </joint>
+  <!--  TODO: Update real gear ratio -->
+  <transmission name="tran1">
+    <type>transmission_interface/SimpleTransmission</type>
+    <joint name="Joint1">
+      <hardwareInterface>hardware_interface/PositionJointInterface</hardwareInterface>
+    </joint>
+    <actuator name="motor_1">
+      <hardwareInterface>hardware_interface/PositionJointInterface</hardwareInterface>
+      <mechanicalReduction>1</mechanicalReduction>
+    </actuator>
+  </transmission>
+  <transmission name="tran2">
+    <type>transmission_interface/SimpleTransmission</type>
+    <joint name="Joint2">
+      <hardwareInterface>hardware_interface/PositionJointInterface</hardwareInterface>
+    </joint>
+    <actuator name="motor_2">
+      <hardwareInterface>hardware_interface/PositionJointInterface</hardwareInterface>
+      <mechanicalReduction>1</mechanicalReduction>
+    </actuator>
+  </transmission>
+  <transmission name="tran3">
+    <type>transmission_interface/SimpleTransmission</type>
+    <joint name="Joint3">
+      <hardwareInterface>hardware_interface/PositionJointInterface</hardwareInterface>
+    </joint>
+    <actuator name="motor_3">
+      <hardwareInterface>hardware_interface/PositionJointInterface</hardwareInterface>
+      <mechanicalReduction>1</mechanicalReduction>
+    </actuator>
+  </transmission>
+  <transmission name="tran4">
+    <type>transmission_interface/SimpleTransmission</type>
+    <joint name="Joint4">
+      <hardwareInterface>hardware_interface/PositionJointInterface</hardwareInterface>
+    </joint>
+    <actuator name="motor_4">
+      <hardwareInterface>hardware_interface/PositionJointInterface</hardwareInterface>
+      <mechanicalReduction>1</mechanicalReduction>
+    </actuator>
+  </transmission>
+  <transmission name="tran5">
+    <type>transmission_interface/SimpleTransmission</type>
+    <joint name="Joint5">
+      <hardwareInterface>hardware_interface/PositionJointInterface</hardwareInterface>
+    </joint>
+    <actuator name="motor_5">
+      <hardwareInterface>hardware_interface/PositionJointInterface</hardwareInterface>
+      <mechanicalReduction>1</mechanicalReduction>
+    </actuator>
+  </transmission>
+  <transmission name="tran6">
+    <type>transmission_interface/SimpleTransmission</type>
+    <joint name="Joint6">
+      <hardwareInterface>hardware_interface/PositionJointInterface</hardwareInterface>
+    </joint>
+    <actuator name="motor_6">
+      <hardwareInterface>hardware_interface/PositionJointInterface</hardwareInterface>
+      <mechanicalReduction>1</mechanicalReduction>
+    </actuator>
+  </transmission>
 </robot>

Commit message: Add joint velocity in urdf to make it movable in Gazebo

File: mini_bot/urdf/mini_bot.urdf.xacro (robot description, xacro)
@@ -1,15 +1,19 @@
 <?xml version="1.0"?>
 <!-- NexCOBOT MiniBOT -->
-<robot name="mini_bot" xmlns:xacro="http://www.ros.org/wiki/xacro">
+<robot name="minibot" xmlns:xacro="http://www.ros.org/wiki/xacro">
   <!-- Constants for robot dimensions -->
   <xacro:property name="PI" value="3.1415926535897931"/>
   <xacro:property name="deg" value="0.017453293"/> <!-- Degrees to Radians -->
-  <xacro:property name="mass0" value="3.0361"/> <!-- assumption value for mass -->
-  <xacro:property name="mass1" value="1.8294"/> <!-- assumption value for mass -->
-  <xacro:property name="mass2" value="1.199"/> <!-- assumption value for mass -->
-  <xacro:property name="mass3" value="0.41277"/> <!-- assumption value for mass -->
-  <xacro:property name="mass4" value="0.34299"/> <!-- assumption value for mass -->
-  <xacro:property name="mass5" value="0.24686"/> <!-- assumption value for mass -->
-  <xacro:property name="mass6" value="0.024508"/> <!-- assumption value for mass -->
+  <!-- assumption value for mass -->
+  <xacro:property name="mass0" value="3.0361"/>
+  <xacro:property name="mass1" value="1.8294"/>
+  <xacro:property name="mass2" value="1.199"/>
+  <xacro:property name="mass3" value="0.41277"/>
+  <xacro:property name="mass4" value="0.34299"/>
+  <xacro:property name="mass5" value="0.24686"/>
+  <xacro:property name="mass6" value="0.024508"/>
+  <!-- Joint velocity and acceleration in degree -->
+  <xacro:property name="vel" value="50"/>
+  <xacro:property name="acc" value="20"/>
   <!-- Import all Gazebo-customization elements, including Gazebo colors -->
   <xacro:include filename="$(find mini_bot)/urdf/mini_bot.gazebo" />
@@ -77,5 +81,5 @@
     <child link="A1_Link" />
     <axis xyz="0 0 1" />
-    <limit lower="-2.617993878" upper="3.019419606" effort="0" velocity="0" />
+    <limit lower="-2.617993878" upper="3.019419606" effort="${acc*deg}" velocity="${vel*deg}" />
     <dynamics damping="0.7"/>
   </joint>
@@ -111,5 +115,5 @@
     <child link="A2_Link" />
     <axis xyz="0 0 1" />
-    <limit lower="-1.6057029118" upper="1.9198621772" effort="0" velocity="0" />
+    <limit lower="-1.6057029118" upper="1.9198621772" effort="${acc*deg}" velocity="${vel*deg}" />
     <dynamics damping="0.7"/>
   </joint>
@@ -144,5 +148,5 @@
     <child link="A3_Link" />
     <axis xyz="0 0 1" />
-    <limit lower="-1.0821041362" upper="2.5307274154" effort="0" velocity="0" />
+    <limit lower="-1.0821041362" upper="2.5307274154" effort="${acc*deg}" velocity="${vel*deg}" />
     <dynamics damping="0.7"/>
   </joint>
@@ -177,5 +181,5 @@
     <child link="A4_Link" />
     <axis xyz="0 0 1" />
-    <limit lower="-2.0943951024" upper="3.0805061298" effort="0" velocity="0" />
+    <limit lower="-2.0943951024" upper="3.0805061298" effort="${acc*deg}" velocity="${vel*deg}" />
     <dynamics damping="0.7"/>
   </joint>
@@ -210,5 +214,5 @@
     <child link="A5_Link" />
     <axis xyz="0 0 1" />
-    <limit lower="-1.8325957146" upper="1.8325957146" effort="0" velocity="0" />
+    <limit lower="-1.8325957146" upper="1.8325957146" effort="${acc*deg}" velocity="${vel*deg}" />
     <dynamics damping="0.7"/>
   </joint>
@@ -243,5 +247,5 @@
     <child link="A6_Link" />
     <axis xyz="0 0 1" />
-    <limit lower="-3.1415926536" upper="3.1415926536" effort="0" velocity="0" />
+    <limit lower="-3.1415926536" upper="3.1415926536" effort="${acc*deg}" velocity="${vel*deg}" />
     <dynamics damping="0.7"/>
   </joint>
